File: schematics/PSLab-GroveShield.sch (KiCad schematic (older format))
At the start: 28 parts, among them J1 I2C G6, J10 I2C G2, J11 I2C G1, J12 SPI G2, J13 ESP, J14 UART G1, J15 External Power, J16 I2C-2, J17 SPI G1, J3 I2C G5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

Commit message: feat: route updates and refactor
Parts:
- removed S1: OpenHardware, Symbols:OSHW-Logo_5.7x6mm_SilkScreen, symbol PSLab:Logos
- removed S10, S3: OpnTec_Logo, Custom_Components:OpnTec_Logo, symbol PSLab:Logos
- removed S4: ESD-Logo, Symbols:ESD-Logo_6.6x6mm_SilkScreen, symbol PSLab:Logos
- removed S5: PSL_Logo, Custom_Components:PSL_Logo, symbol PSLab:Logos
- removed S6: FOSSASIA_Logo_L, Custom_Components:FOSSASIA_LogoL, symbol PSLab:Logos
- removed S7: FOSSASIA_Logo_S, Custom_Components:FOSSASIA_Logo, symbol PSLab:Logos
- removed S8: QR_Code, Custom_Components:Website_QR, symbol PSLab:Logos
- removed S9: PSLabDotIO_B, Custom_Components:PSLabDotIO4000, symbol PSLab:Logos
- S2: symbol PSLab:Logos -> PSLab-GroveShield-rescue:Logos-PSLab
Changed lines of the file:
@@
 +5V
 $Comp
-L PSLab:Logos S?
-U 1 1 5F116DB3
-P 1345 4000
-AR Path="/5C27B0EA/5F116DB3" Ref="S?"  Part="1"
-AR Path="/5F116DB3" Ref="S1"  Part="1"
-F 0 "S1" H 1345 3880 60  0000 C CNN
-F 1 "OpenHardware" H 1345 4120 60  0000 C CNN
-F 2 "Symbols:OSHW-Logo_5.7x6mm_SilkScreen" H 1345 4000 60  0001 C CNN
-F 3 "" H 1345 4000 60  0001 C CNN
-	1    1345 4000
-	1    0    0    -1
-$EndComp
-$Comp
-L PSLab:Logos S?
-U 1 1 5F116DB9
-P 2245 4000
-AR Path="/5C27B0EA/5F116DB9" Ref="S?"  Part="1"
-AR Path="/5F116DB9" Ref="S4"  Part="1"
-F 0 "S4" H 2245 3880 60  0000 C CNN
-F 1 "ESD-Logo" H 2245 4120 60  0000 C CNN
-F 2 "Symbols:ESD-Logo_6.6x6mm_SilkScreen" H 2245 4000 60  0001 C CNN
-F 3 "" H 2245 4000 60  0001 C CNN
-	1    2245 4000
-	1    0    0    -1
-$EndComp
-$Comp
-L PSLab:Logos S?
-U 1 1 5F116DBF
-P 3245 4000
-AR Path="/5C27B0EA/5F116DBF" Ref="S?"  Part="1"
-AR Path="/5F116DBF" Ref="S7"  Part="1"
-F 0 "S7" H 3245 3880 60  0000 C CNN
-F 1 "FOSSASIA_Logo_S" H 3245 4120 60  0000 C CNN
-F 2 "Custom_Components:FOSSASIA_Logo" H 3245 4000 60  0001 C CNN
-F 3 "" H 3245 4000 60  0001 C CNN
-	1    3245 4000
-	1    0    0    -1
-$EndComp
-$Comp
-L PSLab:Logos S?
-U 1 1 5F116DC5
-P 4195 4000
-AR Path="/5C27B0EA/5F116DC5" Ref="S?"  Part="1"
-AR Path="/5F116DC5" Ref="S10"  Part="1"
-F 0 "S10" H 4195 3880 60  0000 C CNN
-F 1 "OpnTec_Logo" H 4195 4120 60  0000 C CNN
-F 2 "Custom_Components:OpnTec_Logo" H 4195 4000 60  0001 C CNN
-F 3 "" H 4195 4000 60  0001 C CNN
-	1    4195 4000
-	1    0    0    -1
-$EndComp
-$Comp
-L PSLab:Logos S?
+L PSLab-GroveShield-rescue:Logos-PSLab S?
 U 1 1 5F116DCB
 P 1855 4670
@@
 	1    0    0    -1
 $EndComp
-$Comp
-L PSLab:Logos S?
-U 1 1 5F116DD1
-P 2750 4675
-AR Path="/5C27B0EA/5F116DD1" Ref="S?"  Part="1"
-AR Path="/5F116DD1" Ref="S5"  Part="1"
-F 0 "S5" H 2750 4555 60  0000 C CNN
-F 1 "PSL_Logo" H 2750 4795 60  0000 C CNN
-F 2 "Custom_Components:PSL_Logo" H 2750 4675 60  0001 C CNN
-F 3 "" H 2750 4675 60  0001 C CNN
-	1    2750 4675
-	1    0    0    -1
-$EndComp
-$Comp
-L PSLab:Logos S?
-U 1 1 5F116DD7
-P 3700 4675
-AR Path="/5C27B0EA/5F116DD7" Ref="S?"  Part="1"
-AR Path="/5F116DD7" Ref="S8"  Part="1"
-F 0 "S8" H 3700 4555 60  0000 C CNN
-F 1 "QR_Code" H 3700 4795 60  0000 C CNN
-F 2 "Custom_Components:Website_QR" H 3700 4675 60  0001 C CNN
-F 3 "" H 3700 4675 60  0001 C CNN
-	1    3700 4675
-	1    0    0    -1
-$EndComp
-$Comp
-L PSLab:Logos S?
-U 1 1 5F116DDD
-P 1865 5350
-AR Path="/5C27B0EA/5F116DDD" Ref="S?"  Part="1"
-AR Path="/5F116DDD" Ref="S3"  Part="1"
-F 0 "S3" H 1865 5230 60  0000 C CNN
-F 1 "OpnTec_Logo" H 1865 5470 60  0000 C CNN
-F 2 "Custom_Components:OpnTec_Logo" H 1865 5350 60  0001 C CNN
-F 3 "" H 1865 5350 60  0001 C CNN
-	1    1865 5350
-	1    0    0    -1
-$EndComp
-$Comp
-L PSLab:Logos S?
-U 1 1 5F116DE3
-P 2765 5350
-AR Path="/5C27B0EA/5F116DE3" Ref="S?"  Part="1"
-AR Path="/5F116DE3" Ref="S6"  Part="1"
-F 0 "S6" H 2765 5230 60  0000 C CNN
-F 1 "FOSSASIA_Logo_L" H 2765 5470 60  0000 C CNN
-F 2 "Custom_Components:FOSSASIA_LogoL" H 2765 5350 60  0001 C CNN
-F 3 "" H 2765 5350 60  0001 C CNN
-	1    2765 5350
-	1    0    0    -1
-$EndComp
-$Comp
-L PSLab:Logos S?
-U 1 1 5F116DE9
-P 3705 5340
-AR Path="/5C27B0EA/5F116DE9" Ref="S?"  Part="1"
-AR Path="/5F116DE9" Ref="S9"  Part="1"
-F 0 "S9" H 3705 5220 60  0000 C CNN
-F 1 "PSLabDotIO_B" H 3705 5460 60  0000 C CNN
-F 2 "Custom_Components:PSLabDotIO4000" H 3705 5340 60  0001 C CNN
-F 3 "" H 3705 5340 60  0001 C CNN
-	1    3705 5340
-	1    0    0    -1
-$EndComp
